File: Project_Files/coupling_board_kicad/coupling_board_v3/Kicad-project/DSUB_ADCIO_adapter/DSUB_ADCIO_adapter.kicad_pcb (KiCad board)
At the start: 2 copper layers, 36.1 x 70 mm, 6 parts, among them J1 Conn_02x04_Odd_Even, J10 Conn_02x12_Odd_Even, J2 Conn_02x04_Odd_Even, J3 Conn_02x04_Odd_Even, J5 Conn_02x12_Odd_Even, J6 DB25_Socket

Commit message: Random commit
Parts:
- removed J10: Conn_02x12_Odd_Even, Connector_PinHeader_2.54mm:PinHeader_2x12_P2.54mm_Vertical
- added J4: Conn_02x12_Odd_Even, Connector_PinHeader_2.54mm:PinHeader_2x12_P2.54mm_Vertical, B.Cu at (143.5, 95.5)
Routing:
- net 3V3_VCUT: track 30.7 -> 98.6 mm, vias 1 -> 0
- net GND1: track 15.9 -> 63.9 mm, vias 7 -> 27
- net /ADC_08: track 48.2 -> 19.8 mm
- net /ADC_18: track 45.8 -> 21.2 mm
- net /ADC_09: track 41.8 -> 19.0 mm
- net /ADC_19: track 45.4 -> 27.4 mm
- net VDD_VCUT: track 46.2 -> 50.3 mm
