File: Project_Files/coupling_board_kicad/coupling_board_v3/Kicad-project/DSUB_ADCIO_adapter/DSUB_ADCIO_adapter.kicad_sch (KiCad schematic)
At the start: 6 parts, among them J1 Conn_02x04_Odd_Even, J10 Conn_02x12_Odd_Even, J2 Conn_02x04_Odd_Even, J3 Conn_02x04_Odd_Even, J4 Conn_02x12_Odd_Even, J6 DB25_Socket

Commit message: Fixed adcio coupler
Parts:
- removed J4: Conn_02x12_Odd_Even, Connector_PinHeader_2.54mm:PinHeader_2x12_P2.54mm_Vertical, symbol Connector_Generic:Conn_02x12_Odd_Even
- added J5: Conn_02x12_Odd_Even, Connector_PinHeader_2.54mm:PinHeader_2x12_P2.54mm_Vertical, symbol Connector_Generic:Conn_02x12_Odd_Even
Connections:
- net ADC_00: now also J5.2 (Pin_2)
- net ADC_01: now also J5.4 (Pin_4)
- net ADC_02: now also J5.8 (Pin_8)
- net ADC_03: now also J5.10 (Pin_10)
- net ADC_14: now also J5.15 (Pin_15)
- net ADC_18: now also J2.3 (Pin_3); no longer J2.1 (Pin_1)
- net ADC_19: now also J2.1 (Pin_1); no longer J2.3 (Pin_3)
- net GND1: now also J5.1 (Pin_1), J5.12 (Pin_12), J5.13 (Pin_13), J5.18 (Pin_18), J5.19 (Pin_19), J5.24 (Pin_24), J5.6 (Pin_6), J5.7 (Pin_7)
- net vcut_COPI: now also J5.11 (Pin_11)
- net vcut_CS: now also J5.20 (Pin_20)
- net vcut_S0: now also J5.21 (Pin_21)
- net vcut_S1: now also J5.23 (Pin_23)
- net vcut_S2: now also J5.22 (Pin_22)
- net vcut_S3: now also J5.16 (Pin_16)
- net vcut_S4: now also J5.14 (Pin_14)
- net vcut_SCLK: now also J5.17 (Pin_17)
- net vcut_~{CLR}: now also J5.9 (Pin_9)
- net vcut_~{LDAC}: now also J5.3 (Pin_3)
- net vcut_~{RESET}: now also J5.5 (Pin_5)
Changed lines of the file:
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@@
-	(wire
-		(pts
-			(xy 95.25 73.66) (xy 102.87 73.66)
-		)
-		(stroke
-			(width 0)
-			(type default)
-		)
-	)
 	(wire
 		(pts
@@
 		)
 	)
-	(label "ADC_18"
+	(label "ADC_19"
 		(at 41.91 57.15 0)
 		(effects
@@
 		)
 	)
-	(label "ADC_01"
-		(at 95.25 73.66 0)
-		(effects
-			(font
-				(size 1.27 1.27)
-			)
-			(justify left bottom)
-		)
-	)
 	(label "vcut_~{RESET}"
 		(at 175.26 111.76 0)
@@
 		)
 	)
-	(label "ADC_19"
+	(label "ADC_18"
 		(at 41.91 59.69 0)
 		(effects
@@
 	)
 	(symbol
-		(lib_id "Connector_Generic:Conn_02x12_Odd_Even")
-		(at 58.42 102.87 0)
-		(unit 1)
-		(exclude_from_sim no)
-		(in_bom yes)
-		(on_board yes)
-		(dnp no)
-		(property "Reference" "J4"
-			(at 59.69 83.82 0)
-			(effects
-				(font
-					(size 1.27 1.27)
-				)
-			)
-		)
-		(property "Value" "Conn_02x12_Odd_Even"
-			(at 59.69 86.36 0)
-			(effects
-				(font
-					(size 1.27 1.27)
-				)
-			)
-		)
-		(property "Footprint" "Connector_PinHeader_2.54mm:PinHeader_2x12_P2.54mm_Vertical"
-			(at 58.42 102.87 0)
-			(effects
-				(font
-					(size 1.27 1.27)
-				)
-				(hide yes)
-			)
-		)
-		(property "Datasheet" "~"
-			(at 58.42 102.87 0)
-			(effects
-				(font
-					(size 1.27 1.27)
-				)
-				(hide yes)
-			)
-		)
-		(property "Description" "Generic connector, double row, 02x12, odd/even pin numbering scheme (row 1 odd numbers, row 2 even numbers), script generated (kicad-library-utils/schlib/autogen/connector/)"
-			(at 58.42 102.87 0)
-			(effects
-				(font
-					(size 1.27 1.27)
-				)
-				(hide yes)
-			)
-		)
-		(property "JLCPCB Part #" "C132440"
-			(at 58.42 102.87 0)
-			(effects
-				(font
-					(size 1.27 1.27)
-				)
-				(hide yes)
-			)
-		)
-		(property "JLCPCB Rotation Offset" "-90"
-			(at 58.42 102.87 0)
-			(effects
-				(font
-					(size 1.27 1.27)
-				)
-				(hide yes)
-			)
-		)
-		(property "JLCPCB Position Offset" "0.5,0"
-			(at 58.42 102.87 0)
-			(effects
-				(font
-					(size 1.27 1.27)
-				)
-				(hide yes)
-			)
-		)
-		(pin "1"
-		)
-		(pin "10"
-		)
-		(pin "11"
-		)
-		(pin "12"
-		)
-		(pin "13"
-		)
-		(pin "14"
-		)
-		(pin "15"
-		)
-		(pin "16"
-		)
-		(pin "17"
-		)
-		(pin "18"
-		)
-		(pin "19"
-		)
-		(pin "2"
-		)
-		(pin "20"
-		)
-		(pin "21"
-		)
-		(pin "22"
-		)
-		(pin "23"
-		)
-		(pin "24"
-		)
-		(pin "3"
-		)
-		(pin "4"
-		)
-		(pin "5"
-		)
-		(pin "6"
-		)
-		(pin "7"
-		)
-		(pin "8"
-		)
-		(pin "9"
-		)
-		(instances
-			(project "DSUB_ADCIO_adapter"
-				(path "/1aa7e185-a043-4a74-ab54-212e9cb98b06"
-					(reference "J4")
-					(unit 1)
-				)
-			)
-		)
-	)
-	(symbol
 		(lib_id "power:GND")
 		(at 72.39 67.31 0)
@@
 					(unit 1)
 				)
+			)
+		)
+	)
+	(symbol
+		(lib_id "Connector_Generic:Conn_02x12_Odd_Even")
+		(at 60.96 102.87 0)
+		(mirror y)
+		(unit 1)
+		(exclude_from_sim no)
+		(in_bom yes)
+		(on_board yes)
+		(dnp no)
+		(property "Reference" "J5"
+			(at 59.69 83.82 0)
+			(effects
+				(font
+					(size 1.27 1.27)
+				)
+			)
+		)
+		(property "Value" "Conn_02x12_Odd_Even"
+			(at 59.69 86.36 0)
+			(effects
+				(font
+					(size 1.27 1.27)
+				)
+			)
+		)
+		(property "Footprint" "Connector_PinHeader_2.54mm:PinHeader_2x12_P2.54mm_Vertical"
+			(at 60.96 102.87 0)
+			(effects
+				(font
+					(size 1.27 1.27)
+				)
+				(hide yes)
+			)
+		)
+		(property "Datasheet" "~"
+			(at 60.96 102.87 0)
+			(effects
+				(font
+					(size 1.27 1.27)
+				)
+				(hide yes)
+			)
+		)
+		(property "Description" "Generic connector, double row, 02x12, odd/even pin numbering scheme (row 1 odd numbers, row 2 even numbers), script generated (kicad-library-utils/schlib/autogen/connector/)"
+			(at 60.96 102.87 0)
+			(effects
+				(font
+					(size 1.27 1.27)
+				)
+				(hide yes)
+			)
+		)
+		(property "JLCPCB Part #" "C132440"
+			(at 60.96 102.87 0)
+			(effects
+				(font
+					(size 1.27 1.27)
+				)
+				(hide yes)
+			)
+		)
+		(property "JLCPCB Rotation Offset" "-90"
+			(at 60.96 102.87 0)
+			(effects
+				(font
+					(size 1.27 1.27)
+				)
+				(hide yes)
+			)
+		)
+		(property "JLCPCB Position Offset" "0.5,0"
+			(at 60.96 102.87 0)
+			(effects
+				(font
+					(size 1.27 1.27)
+				)
+				(hide yes)
+			)
+		)
+		(pin "1"
+		)
+		(pin "10"
+		)
+		(pin "11"
+		)
+		(pin "12"
+		)
+		(pin "13"
+		)
+		(pin "14"
+		)
+		(pin "15"
+		)
+		(pin "16"
+		)
+		(pin "17"
+		)
+		(pin "18"
+		)
+		(pin "19"
+		)
+		(pin "2"
+		)
+		(pin "20"
+		)
+		(pin "21"
+		)
+		(pin "22"
+		)
+		(pin "23"
+		)
+		(pin "24"
+		)
+		(pin "3"
+		)
+		(pin "4"
+		)
+		(pin "5"
+		)
+		(pin "6"
+		)
+		(pin "7"
+		)
+		(pin "8"
+		)
+		(pin "9"
+		)
+		(instances
+			(project "DSUB_ADCIO_adapter"
+				(path "/1aa7e185-a043-4a74-ab54-212e9cb98b06"
+					(reference "J5")
+					(unit 1)
+				)

Commit message: Random commit
Parts:
- removed J10: Conn_02x12_Odd_Even, Connector_PinHeader_2.54mm:PinHeader_2x12_P2.54mm_Vertical, symbol Connector_Generic:Conn_02x12_Odd_Even
- added J4: Conn_02x12_Odd_Even, Connector_PinHeader_2.54mm:PinHeader_2x12_P2.54mm_Vertical, symbol Connector_Generic:Conn_02x12_Odd_Even
Connections:
- net 3V3_VCUT: now also J4.22 (Pin_22), J4.24 (Pin_24)
- net ADC_08: now also J4.2 (Pin_2)
- net ADC_09: now also J4.4 (Pin_4)
- net ADC_18: now also J4.3 (Pin_3)
- net ADC_19: now also J4.5 (Pin_5)
- net GND1: now also J4.1 (Pin_1), J4.13 (Pin_13), J4.15 (Pin_15), J4.17 (Pin_17), J4.18 (Pin_18), J4.19 (Pin_19), J4.20 (Pin_20)
- net VDD_VCUT: now also J4.14 (Pin_14), J4.16 (Pin_16)
Changed lines of the file:
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@@
 	)
 	(no_connect
-		(at 118.11 96.52)
+		(at 119.38 96.52)
 	)
 	(no_connect
-		(at 118.11 99.06)
+		(at 119.38 99.06)
 	)
 	(no_connect
-		(at 130.81 104.14)
+		(at 132.08 104.14)
 	)
 	(no_connect
-		(at 130.81 119.38)
+		(at 132.08 119.38)
 	)
 	(no_connect
@@
 	)
 	(no_connect
-		(at 130.81 116.84)
+		(at 132.08 116.84)
 	)
 	(no_connect
@@
 	)
 	(no_connect
-		(at 130.81 99.06)
+		(at 132.08 99.06)
 	)
 	(no_connect
-		(at 118.11 101.6)
+		(at 119.38 101.6)
 	)
 	(no_connect
-		(at 130.81 101.6)
+		(at 132.08 101.6)
 	)
 	(no_connect
-		(at 118.11 104.14)
+		(at 119.38 104.14)
 	)
 	(no_connect
@@
 	(wire
 		(pts
-			(xy 118.11 116.84) (xy 106.68 116.84)
+			(xy 119.38 116.84) (xy 106.68 116.84)
 		)
 		(stroke
@@
 	(wire
 		(pts
-			(xy 148.59 109.22) (xy 130.81 109.22)
+			(xy 148.59 109.22) (xy 132.08 109.22)
 		)
 		(stroke
@@
 	(wire
 		(pts
-			(xy 138.43 96.52) (xy 130.81 96.52)
+			(xy 138.43 96.52) (xy 132.08 96.52)
 		)
 		(stroke
@@
 	(wire
 		(pts
-			(xy 118.11 114.3) (xy 101.6 114.3)
+			(xy 119.38 114.3) (xy 101.6 114.3)
 		)
 		(stroke
@@
 	(wire
 		(pts
-			(xy 138.43 93.98) (xy 130.81 93.98)
-		)
-		(stroke
-			(width 0)
-			(type default)
-		)
-	)
-	(wire
-		(pts
-			(xy 148.59 114.3) (xy 130.81 114.3)
+			(xy 138.43 93.98) (xy 132.08 93.98)
+		)
+		(stroke
+			(width 0)
+			(type default)
+		)
+	)
+	(wire
+		(pts
+			(xy 148.59 114.3) (xy 132.08 114.3)
 		)
 		(stroke
@@
 	(wire
 		(pts
-			(xy 118.11 111.76) (xy 101.6 111.76)
-		)
-		(stroke
-			(width 0)
-			(type default)
-		)
-	)
-	(wire
-		(pts
-			(xy 118.11 119.38) (xy 106.68 119.38)
+			(xy 119.38 111.76) (xy 101.6 111.76)
+		)
+		(stroke
+			(width 0)
+			(type default)
+		)
+	)
+	(wire
+		(pts
+			(xy 119.38 119.38) (xy 106.68 119.38)
 		)
 		(stroke
@@
 	(wire
 		(pts
-			(xy 148.59 106.68) (xy 130.81 106.68)
+			(xy 148.59 106.68) (xy 132.08 106.68)
 		)
 		(stroke
@@
 	(wire
 		(pts
-			(xy 148.59 91.44) (xy 130.81 91.44)
-		)
-		(stroke
-			(width 0)
-			(type default)
-		)
-	)
-	(wire
-		(pts
-			(xy 118.11 109.22) (xy 111.76 109.22)
-		)
-		(stroke
-			(width 0)
-			(type default)
-		)
-	)
-	(wire
-		(pts
-			(xy 118.11 106.68) (xy 111.76 106.68)
+			(xy 148.59 91.44) (xy 132.08 91.44)
+		)
+		(stroke
+			(width 0)
+			(type default)
+		)
+	)
+	(wire
+		(pts
+			(xy 119.38 109.22) (xy 111.76 109.22)
+		)
+		(stroke
+			(width 0)
+			(type default)
+		)
+	)
+	(wire
+		(pts
+			(xy 119.38 106.68) (xy 111.76 106.68)
 		)
 		(stroke
@@
 	(wire
 		(pts
-			(xy 118.11 93.98) (xy 110.49 93.98)
+			(xy 119.38 93.98) (xy 110.49 93.98)
 		)
 		(stroke
@@
 	(wire
 		(pts
-			(xy 118.11 91.44) (xy 110.49 91.44)
+			(xy 119.38 91.44) (xy 110.49 91.44)
 		)
 		(stroke
@@
 	(wire
 		(pts
-			(xy 148.59 111.76) (xy 130.81 111.76)
+			(xy 148.59 111.76) (xy 132.08 111.76)
 		)
 		(stroke
@@
 	)
 	(symbol
+		(lib_id "Connector_Generic:Conn_02x12_Odd_Even")
+		(at 127 104.14 0)
+		(mirror y)
+		(unit 1)
+		(exclude_from_sim no)
+		(in_bom yes)
+		(on_board yes)
+		(dnp no)
+		(property "Reference" "J4"
+			(at 125.73 85.09 0)
+			(effects
+				(font
+					(size 1.27 1.27)
+				)
+			)
+		)
+		(property "Value" "Conn_02x12_Odd_Even"
+			(at 125.73 87.63 0)
+			(effects
+				(font
+					(size 1.27 1.27)
+				)
+			)
+		)
+		(property "Footprint" "Connector_PinHeader_2.54mm:PinHeader_2x12_P2.54mm_Vertical"
+			(at 127 104.14 0)
+			(effects
+				(font
+					(size 1.27 1.27)
+				)
+				(hide yes)
+			)
+		)
+		(property "Datasheet" "~"
+			(at 127 104.14 0)
+			(effects
+				(font
+					(size 1.27 1.27)
+				)
+				(hide yes)
+			)
+		)
+		(property "Description" "Generic connector, double row, 02x12, odd/even pin numbering scheme (row 1 odd numbers, row 2 even numbers), script generated (kicad-library-utils/schlib/autogen/connector/)"
+			(at 127 104.14 0)
+			(effects
+				(font
+					(size 1.27 1.27)
+				)
+				(hide yes)
+			)
+		)
+		(property "JLCPCB Part #" "C132440"
+			(at 127 104.14 0)
+			(effects
+				(font
+					(size 1.27 1.27)
+				)
+				(hide yes)
+			)
+		)
+		(property "JLCPCB Rotation Offset" "-90"
+			(at 127 104.14 0)
+			(effects
+				(font
+					(size 1.27 1.27)
+				)
+				(hide yes)
+			)
+		)
+		(property "JLCPCB Position Offset" "0.5,0"
+			(at 127 104.14 0)
+			(effects
+				(font
+					(size 1.27 1.27)
+				)
+				(hide yes)
+			)
+		)
+		(pin "1"
+		)
+		(pin "10"
+		)
+		(pin "11"
+		)
+		(pin "12"
+		)
+		(pin "13"
+		)
+		(pin "14"
+		)
+		(pin "15"
+		)
+		(pin "16"
+		)
+		(pin "17"
+		)
+		(pin "18"
+		)
+		(pin "19"
+		)
+		(pin "2"
+		)
+		(pin "20"
+		)
+		(pin "21"
+		)
+		(pin "22"
+		)
+		(pin "23"
+		)
+		(pin "24"
+		)
+		(pin "3"
+		)
+		(pin "4"
+		)
+		(pin "5"
+		)
+		(pin "6"
+		)
+		(pin "7"
+		)
+		(pin "8"
+		)
+		(pin "9"
+		)
+		(instances
+			(project "DSUB_ADCIO_adapter"
+				(path "/1aa7e185-a043-4a74-ab54-212e9cb98b06"
+					(reference "J4")
+					(unit 1)
+				)
+			)
+		)
+	)
+	(symbol
 		(lib_id "power:GND")
 		(at 72.39 67.31 0)
@@
 					(unit 1)
 				)
-			)
-		)
-	)
-	(symbol
-		(lib_id "Connector_Generic:Conn_02x12_Odd_Even")
-		(at 123.19 104.14 0)
-		(unit 1)
-		(exclude_from_sim no)
-		(in_bom yes)
-		(on_board yes)
-		(dnp no)
-		(property "Reference" "J10"
-			(at 124.46 85.09 0)
-			(effects
-				(font
-					(size 1.27 1.27)
-				)
-			)
-		)
-		(property "Value" "Conn_02x12_Odd_Even"
-			(at 124.46 87.63 0)
-			(effects
-				(font
-					(size 1.27 1.27)
-				)
-			)
-		)
-		(property "Footprint" "Connector_PinHeader_2.54mm:PinHeader_2x12_P2.54mm_Vertical"
-			(at 123.19 104.14 0)
-			(effects
-				(font
-					(size 1.27 1.27)
-				)
-				(hide yes)
-			)
-		)
-		(property "Datasheet" "~"
-			(at 123.19 104.14 0)
-			(effects
-				(font
-					(size 1.27 1.27)
-				)
-				(hide yes)
-			)
-		)
-		(property "Description" "Generic connector, double row, 02x12, odd/even pin numbering scheme (row 1 odd numbers, row 2 even numbers), script generated (kicad-library-utils/schlib/autogen/connector/)"
-			(at 123.19 104.14 0)
-			(effects
-				(font
-					(size 1.27 1.27)
-				)
-				(hide yes)
-			)
-		)
-		(property "JLCPCB Part #" "C132440"
-			(at 123.19 104.14 0)
-			(effects
-				(font
-					(size 1.27 1.27)
-				)
-				(hide yes)
-			)
-		)
-		(property "JLCPCB Rotation Offset" "-90"
-			(at 123.19 104.14 0)
-			(effects
-				(font
-					(size 1.27 1.27)
-				)
-				(hide yes)
-			)
-		)
-		(property "JLCPCB Position Offset" "0.5,0"
-			(at 123.19 104.14 0)
-			(effects
-				(font
-					(size 1.27 1.27)
-				)
-				(hide yes)
-			)
-		)
-		(pin "1"
-		)
-		(pin "10"
-		)
-		(pin "11"
-		)
-		(pin "12"
-		)
-		(pin "13"
-		)
-		(pin "14"
-		)
-		(pin "15"
-		)
-		(pin "16"
-		)
-		(pin "17"
-		)
-		(pin "18"
-		)
-		(pin "19"
-		)
-		(pin "2"
-		)
-		(pin "20"
-		)
-		(pin "21"
-		)
-		(pin "22"
-		)
-		(pin "23"
-		)
-		(pin "24"
-		)
-		(pin "3"
-		)
-		(pin "4"
-		)
-		(pin "5"
-		)
-		(pin "6"
-		)
-		(pin "7"
-		)
-		(pin "8"
-		)
-		(pin "9"
-		)
-		(instances
-			(project "DSUB_ADCIO_adapter"
-				(path "/1aa7e185-a043-4a74-ab54-212e9cb98b06"
-					(reference "J10")
-					(unit 1)
-				)
